File: QASS_PCB/QASS_PCB.kicad_pcb (KiCad board)
At the start: 2 copper layers, 89 parts, among them U2 Seeeduino Xiao rp2040

Commit message: working on it
Parts:
- removed D20, D21, D22, D23, D24, D25, D26, D27, D28, D29, D30, D31, D32, D33, D34, D35, D36, D37, D38, D39: D_Small, Diode_SMD:D_SOD-123
- removed U2: Seeeduino Xiao rp2040, PCM_marbastlib-xp-promicroish:Xiao_rp2040_ACH
- added D40: BAV70_Small, Package_TO_SOT_SMD:SOT-23, B.Cu at (42.9, 37.3)
- added J1: Conn_01x02_Pin, Connector_PinHeader_2.54mm:PinHeader_1x02_P2.54mm_Vertical, B.Cu at (129.9, 19.4)
- added U1: ~, Einzelne Custom:Miao, B.Cu at (128.6, 28.0)
- D1, D10, D11, D12, D13, D14, D15, D16, D17, D18, D19, D2, D3, D4, D5, D6, D7, D8, D9: value D_Small -> BAV70_Small; footprint Diode_SMD:D_SOD-123 -> Package_TO_SOT_SMD:SOT-23
- moved D10 157.7 mm to (57.1, 75.4), turned to -90 degrees
- moved D11 144.2 mm to (95.0, 75.4), turned to -90 degrees
- moved D14 132.3 mm to (209.6, 75.4), turned to -90 degrees
- moved D13 113.5 mm to (171.3, 75.4), turned to -90 degrees
- moved MX41 104.8 mm to (105.2, 130.6)
- moved MX42 102.4 mm to (126.6, 130.2)
- moved D4 101.4 mm to (195.3, 37.3), turned to -90 degrees
- moved D12 97.5 mm to (133.3, 75.4), turned to -90 degrees
- moved D3 82.4 mm to (157.2, 37.3), turned to -90 degrees
- moved D5 70.6 mm to (45.9, 52.4), turned to -90 degrees
- moved D15 67.3 mm to (56.8, 102.4), turned to -90 degrees
- moved D19 64.7 mm to (238.1, 35.7), turned to -90 degrees
- moved MX39 56.8 mm to (219.1, 86.9)
- moved D16 56.2 mm to (96.0, 101.6), turned to -90 degrees
- moved D2 55.9 mm to (111.5, 37.3), turned to -90 degrees
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Connections:
- D1 pad 1: r0 -> Net-(D1-A1)
- D1 pad 2: Net-(D1-A) -> Net-(D1-A2)
- D10 pad 1: r0 -> Net-(D10-A1)
- D10 pad 2: Net-(D10-A) -> Net-(D10-A2)
- D11 pad 1: r0 -> Net-(D11-A1)
- D11 pad 2: Net-(D11-A) -> Net-(D11-A2)
- D12 pad 1: r1 -> Net-(D12-A1)
- D12 pad 2: Net-(D12-A) -> Net-(D12-A2)
- D13 pad 1: r1 -> Net-(D13-A1)
- D13 pad 2: Net-(D13-A) -> Net-(D13-A2)
- D14 pad 1: r1 -> Net-(D14-A1)
- D14 pad 2: Net-(D14-A) -> Net-(D14-A2)
- D15 pad 1: r1 -> Net-(D15-A1)
- D15 pad 2: Net-(D15-A) -> Net-(D15-A2)
- D16 pad 1: r1 -> Net-(D16-A1)
- D16 pad 2: Net-(D16-A) -> Net-(D16-A2)
- D17 pad 1: r1 -> Net-(D17-A1)
- D17 pad 2: Net-(D17-A) -> Net-(D17-A2)
- D18 pad 1: r1 -> Net-(D18-A1)
- D18 pad 2: Net-(D18-A) -> Net-(D18-A2)
- D19 pad 1: r1 -> unconnected-(D19-A1-Pad1)
- D19 pad 2: Net-(D19-A) -> Net-(D19-A2)
- D2 pad 1: r0 -> Net-(D2-A1)
- D2 pad 2: Net-(D2-A) -> Net-(D2-A2)
- D3 pad 1: r0 -> Net-(D3-A1)
- D3 pad 2: Net-(D3-A) -> Net-(D3-A2)
- D4 pad 1: r0 -> Net-(D4-A1)
- D4 pad 2: Net-(D4-A) -> Net-(D4-A2)
- D5 pad 1: r0 -> Net-(D5-A1)
- D5 pad 2: Net-(D5-A) -> Net-(D5-A2)
- D6 pad 1: r0 -> Net-(D6-A1)
- D6 pad 2: Net-(D6-A) -> Net-(D6-A2)
- D7 pad 1: r0 -> Net-(D7-A1)
- D7 pad 2: Net-(D7-A) -> Net-(D7-A2)
- D8 pad 1: r0 -> Net-(D8-A1)
- D8 pad 2: Net-(D8-A) -> Net-(D8-A2)
- D9 pad 1: r0 -> Net-(D9-A1)
- D9 pad 2: Net-(D9-A) -> Net-(D9-A2)
- MX1 pad 2: Net-(D1-A) -> Net-(D40-A1)
- MX10 pad 1: c9 -> Net-(D4-A2)
- MX10 pad 2: Net-(D10-A) -> c9
- MX11 pad 1: c10 -> c9
- MX11 pad 2: Net-(D11-A) -> Net-(D19-A2)
- MX12 pad 2: Net-(D12-A) -> Net-(D5-A1)
- MX13 pad 1: c1 -> Net-(D5-A2)
- MX13 pad 2: Net-(D13-A) -> c1
- MX14 pad 2: Net-(D14-A) -> Net-(D6-A1)
- MX15 pad 1: c3 -> Net-(D6-A2)
- MX15 pad 2: Net-(D15-A) -> c3
- MX16 pad 2: Net-(D16-A) -> Net-(D7-A1)
- MX17 pad 1: c5 -> Net-(D7-A2)
- MX17 pad 2: Net-(D17-A) -> c5
- MX18 pad 2: Net-(D18-A) -> Net-(D8-A1)
- MX19 pad 1: c7 -> Net-(D8-A2)
- MX19 pad 2: Net-(D19-A) -> c7
- MX2 pad 1: c1 -> Net-(D40-A2)
- MX2 pad 2: Net-(D2-A) -> c1
- MX20 pad 2: Net-(D20-A) -> Net-(D9-A1)
- MX21 pad 1: c9 -> Net-(D9-A2)
- MX21 pad 2: Net-(D21-A) -> c9
- MX22 pad 2: Net-(D22-A) -> Net-(D10-A1)
- MX23 pad 1: c1 -> Net-(D10-A2)
- MX23 pad 2: Net-(D23-A) -> c1
- MX24 pad 2: Net-(D24-A) -> Net-(D11-A1)
- MX25 pad 1: c3 -> Net-(D11-A2)
- MX25 pad 2: Net-(D25-A) -> c3
- MX26 pad 2: Net-(D26-A) -> Net-(D12-A1)
- MX27 pad 1: c5 -> Net-(D12-A2)
- MX27 pad 2: Net-(D27-A) -> c5
- MX28 pad 2: Net-(D28-A) -> Net-(D13-A1)
- MX29 pad 1: c7 -> Net-(D13-A2)
- MX29 pad 2: Net-(D29-A) -> c7
- MX3 pad 2: Net-(D3-A) -> Net-(D1-A1)
- MX30 pad 2: Net-(D30-A) -> Net-(D14-A1)
- MX31 pad 1: c9 -> Net-(D14-A2)
- MX31 pad 2: Net-(D31-A) -> c9
- MX32 pad 2: Net-(D32-A) -> Net-(D15-A1)
- MX33 pad 1: c2 -> Net-(D15-A2)
- MX33 pad 2: Net-(D33-A) -> c2
- MX34 pad 2: Net-(D34-A) -> Net-(D16-A1)
- MX35 pad 1: c4 -> Net-(D16-A2)
- MX35 pad 2: Net-(D35-A) -> c4
- MX36 pad 2: Net-(D36-A) -> Net-(D17-A1)
- MX37 pad 1: c6 -> Net-(D17-A2)
- MX37 pad 2: Net-(D37-A) -> c6
- MX38 pad 2: Net-(D38-A) -> Net-(D18-A1)
- MX39 pad 1: c8 -> Net-(D18-A2)
- MX39 pad 2: Net-(D39-A) -> c8
- MX4 pad 1: c3 -> Net-(D1-A2)
- MX4 pad 2: Net-(D4-A) -> c3
- MX40 pad 1: c6 -> Net-(D16-A2)
- MX40 pad 2: Net-(D37-A) -> c4
- MX41 pad 1: c4 -> c5
- MX41 pad 2: Net-(D35-A) -> Net-(D17-A1)
- MX42 pad 2: Net-(D36-A) -> Net-(D17-A1)
- MX5 pad 2: Net-(D5-A) -> Net-(D2-A1)
- MX6 pad 1: c5 -> Net-(D2-A2)
- MX6 pad 2: Net-(D6-A) -> c5
- MX7 pad 2: Net-(D7-A) -> Net-(D3-A1)
- MX8 pad 1: c7 -> Net-(D3-A2)
- MX8 pad 2: Net-(D8-A) -> c7
- MX9 pad 2: Net-(D9-A) -> Net-(D4-A1)

Commit message: Routing down, pretty close to final
Parts:
- added REF**: Clacktales_9mm_whiteSilk, single:Clacktales_9mm_whiteSilk, B.Cu at (63.8, 56.8)
- added Ref**: Val**, single:QASS without text, B.Cu at (205.5, 50.3)
- added Ref**: Val**, single:drawing, B.Cu at (53.9, 57.1)
- S7: footprint PCM_marbastlib-mx:STAB_MX_P_7u -> PCM_marbastlib-mx:STAB_MX_P_10u
- moved D18 58.9 mm to (209.6, 76.2), turned to 90 degrees
- moved MX40 54.9 mm to (114.3, 86.9)
- moved MX41 52.0 mm to (133.3, 86.9)
- moved D17 51.1 mm to (169.9, 76.2), turned to 90 degrees
- moved MX42 50.4 mm to (152.4, 86.9)
- moved MX35 28.6 mm to (104.8, 86.9)
- moved D15 25.8 mm to (57.1, 76.6), turned to 90 degrees
- moved D16 25.0 mm to (95.2, 76.6), turned to 90 degrees
- moved D19 22.3 mm to (215.9, 37.3)
- moved S3 19.0 mm to (104.8, 86.9)
- moved D14 13.1 mm to (209.6, 62.3), turned to 90 degrees
- moved D9 12.7 mm to (202.8, 39.3), turned to 90 degrees
- moved MX36 9.53 mm to (161.9, 86.9)
- moved D11 5.16 mm to (95.2, 70.2)
- moved D13 5.16 mm to (171.4, 70.2)
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Connections:
- D14 pad 3: r2 -> r4
- D19 pad 3: r3 -> r4
- D4 pad 3: r0 -> r4
- D9 pad 3: r1 -> r4
- J1 pad 1: unconnected-(J1-Pin_1-Pad1) -> c0
- J1 pad 2: unconnected-(J1-Pin_2-Pad2) -> c7
- MX10 pad 2: c9 -> c6
- MX11 pad 1: c9 -> c7
- MX20 pad 1: c8 -> c4
- MX21 pad 2: c9 -> c2
- MX30 pad 1: c8 -> c3
- MX31 pad 2: c9 -> c1
- MX32 pad 1: c1 -> c0
- MX33 pad 2: c2 -> c1
- MX34 pad 1: c3 -> c2
- MX35 pad 2: c4 -> c3
- MX36 pad 1: c5 -> c4
- MX37 pad 2: c6 -> c5
- MX38 pad 1: c7 -> c6
- MX39 pad 2: c8 -> c7
- MX40 pad 2: c4 -> c3
- MX41 pad 1: c5 -> c4
- MX42 pad 1: c5 -> c4
- MX9 pad 1: c8 -> c5
- U1 pad 1: unconnected-(U1-P3.2-Pad1) -> c6
- U1 pad 10: unconnected-(U1-P1.6-Pad10) -> c5
- U1 pad 11: unconnected-(U1-P1.5-Pad11) -> c4
- U1 pad 17: unconnected-(U1-P1.0-Pad17) -> c0
- U1 pad 18: unconnected-(U1-P3.3-Pad18) -> c7
- U1 pad 2: unconnected-(U1-P1.1-Pad2) -> r0
- U1 pad 3: unconnected-(U1-P1.2-Pad3) -> r1
- U1 pad 4: unconnected-(U1-P1.3-Pad4) -> c1
- U1 pad 5: unconnected-(U1-P3.5-Pad5) -> c2
- U1 pad 6: unconnected-(U1-P3.4-Pad6) -> c3
- U1 pad 7: unconnected-(U1-P3.1-Pad7) -> r2
- U1 pad 8: unconnected-(U1-RX/CS-Pad8) -> r4
- U1 pad 9: unconnected-(U1-P1.7-Pad9) -> r3
Routing:
- net c1: track 0.00 -> 312.1 mm
- net c2: track 0.00 -> 300.0 mm
- net c3: track 0.00 -> 218.3 mm
- net r3: track 0.00 -> 207.6 mm, vias 0 -> 1
- net c7: track 0.00 -> 195.5 mm
- net c4: track 0.00 -> 192.7 mm
- net c6: track 0.00 -> 171.8 mm
- net c0: track 0.00 -> 169.6 mm
- net r2: track 0.00 -> 157.5 mm, vias 0 -> 1
- net c5: track 0.00 -> 155.7 mm
- net r1: track 0.00 -> 143.2 mm, vias 0 -> 1
- net r0: track 0.00 -> 131.2 mm
- net r4: track 0.00 -> 122.1 mm, vias 0 -> 2
- net Net-(D17-A1): track 0.00 -> 35.1 mm
- net Net-(D19-A2): track 0.00 -> 19.0 mm
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Other:
- board outline added: 219.1 x 80.4 mm
- board text added: "BAE"
- board text added: "BigAssEnter"
- board text added: "Dont solder MCU directly! Use hotswap header or solder switch first."
- board text added: "QASS"
- board text added: "Works with MIAO and XIAO"

Commit message: v1
Parts:
- removed the Ref** at (205.5, 50.3)
- added Ref**: Val**, single:Miaoxiao 10mm, F.Cu at (128.6, 40.1)
- added Ref**: Val**, single:Miaoxiao 10mm, B.Cu at (42.9, 56.8)
- added Ref**: Val**, single:QASS without text wo shadow, B.Cu at (212.5, 48.8)
- MX20: moved to B.Cu
Routing:
- net c2: track 300.0 -> 312.6 mm
- net Net-(D9-A1): track 10.0 -> 17.1 mm
- net c7: track 195.5 -> 191.3 mm
- net c4: track 192.7 -> 191.4 mm
- net Net-(D8-A1): track 8.20 -> 7.19 mm
- net Net-(D6-A1): track 8.20 -> 7.19 mm
- net Net-(D7-A1): track 8.20 -> 7.19 mm
- net Net-(D7-A2): track 5.81 -> 4.82 mm
- net Net-(D6-A2): track 5.81 -> 4.82 mm
- net Net-(D5-A2): track 5.81 -> 4.82 mm
- net Net-(D8-A2): track 5.81 -> 4.82 mm
- net c5: track 155.7 -> 154.7 mm
- net Net-(D15-A1): track 7.72 -> 6.85 mm
- net Net-(D16-A1): track 7.72 -> 6.85 mm
- net Net-(D4-A2): track 11.7 -> 10.9 mm
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Other:
- outline, holes or cut-outs redrawn
- board text added: "https://github.com/Technofrikus/QASS"
- board text added: "v1.0"
- board text removed: "BAE"
- board text removed: "BigAssEnter"
