File: QASS_PCB/QASS_PCB.kicad_pcb (KiCad board)
At the start: 2 copper layers, 219.1 x 80.4 mm, 76 parts, among them J1 Conn_01x02_Pin

Commit message: Added 2.75u right shift option
Parts:
- removed REF**: Clacktales_9mm_whiteSilk, single:Clacktales_9mm_whiteSilk
- removed Ref** (x2): Val**, single:Miaoxiao 10mm
- removed Ref**: Val**, single:QASS without text wo shadow
- removed Ref**: Val**, single:drawing
- added MX43: MX_SW_solder, PCM_marbastlib-mx:SW_MX_1u, F.Cu at (216.7, 67.9)
- added S8: MX_stab, PCM_marbastlib-mx:STAB_MX_2.75u, F.Cu at (216.7, 67.9)
Routing:
- net r3: track 207.0 -> 208.2 mm
- net c1: track 312.1 -> 312.7 mm

Commit message: Added ISO Enter
Parts:
- added ?: , clipboard:06e4d271-3de8-4da3-9581-e3847de2831e, F.Cu at (231.4, 35.7)
- added ?: , clipboard:06e4d271-3de8-4da3-9581-e3847de2831e, F.Cu at (227.8, 27.4)
- added MX44: MX_SW_solder, PCM_marbastlib-mx:SW_MX_1u, F.Cu at (231.0, 39.3)
- added MX45: MX_SW_solder, PCM_marbastlib-mx:SW_MX_1u, F.Cu at (209.6, 48.8)
- added REF**: Clacktales_9mm_whiteSilk, silkscreen:Clacktales_9mm_whiteSilk, B.Cu at (54.5, 55.8)
- added Ref**: Val**, silkscreen:Miaoxiao 10mm, F.Cu at (128.3, 41.1)
- added Ref**: Val**, silkscreen:Miaoxiao 10mm, B.Cu at (44.5, 56.9)
- added Ref**: Val**, silkscreen:QASS without text wo shadow, B.Cu at (207.2, 48.2)
- added Ref**: Val**, silkscreen:Duck 2 with text, B.Cu at (63.7, 56.7)
- added S9: MX_stab, PCM_marbastlib-mx:STAB_MX_P_ISO, F.Cu at (231.0, 39.3)
- MX20: moved to F.Cu
- turned MX11 to 180 degrees
Routing:
- net c7: track 191.3 -> 179.4 mm
- net Net-(D9-A1): track 17.1 -> 10.0 mm
- net Net-(D9-A2): track 16.1 -> 22.5 mm
- net Net-(D19-A2): track 18.6 -> 17.0 mm
- net c2: track 312.6 -> 311.1 mm
- net c4: track 191.4 -> 190.1 mm
- net r4: track 121.4 -> 122.1 mm
Other:
- board text added: "BAE/ANSI"
- board text added: "ISO"

Commit message: Second version added: lowbar
Parts:
- removed the Ref** at (207.2, 48.2)
- added Ref**: Val**, silkscreen:peach simple qass logo, B.Cu at (202.1, 50.6)
Other:
- outline, holes or cut-outs redrawn
- board text added: "Use 3mm high header. Hotswap or solder switch first."
- board text removed: "Dont solder MCU directly! Use hotswap header or solder switch first."
