File: QASS_PCB_Zero_lowbar_Germini/QASS_PCB lowbar.kicad_sch (KiCad schematic)
At the start: 99 parts, among them J2 Conn_01x05_Pin, J3 Conn_01x05_Pin, J4 Conn_01x02_Pin, J5 Conn_01x05_Pin, J6 Conn_01x05_Pin, U2 RP2040-Matrix

Commit message: v1.3 - silkscreen better and one diode orientation more consistent
Parts:
- D1, D10, D11, D12, D13, D14, D15, D16, D17, D18, D19, D2, D20, D21, D22, D23, D24, D25, D26, D27, D28, D29, D3, D30, D31, D32, D33, D34, D35, D36, D37, D38, D39, D4, D5, D6, D7, D8, D9: footprint footprints:Diode-dual -> TFL:Diode-dual
Changed lines of the file:
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@@
 			)
 		)
-		(property "Footprint" "footprints:Diode-dual"
+		(property "Footprint" "TFL:Diode-dual"
 			(at 148.59 88.9 90)
 			(effects
@@
 			)
 		)
-		(property "Footprint" "footprints:Diode-dual"
+		(property "Footprint" "TFL:Diode-dual"
 			(at 158.75 64.77 90)
 			(effects
@@
 			)
 		)
-		(property "Footprint" "footprints:Diode-dual"
+		(property "Footprint" "TFL:Diode-dual"
 			(at 151.13 167.64 90)
 			(effects
@@
 			)
 		)
-		(property "Footprint" "footprints:Diode-dual"
+		(property "Footprint" "TFL:Diode-dual"
 			(at 189.23 88.9 90)
 			(effects
@@
 			)
 		)
-		(property "Footprint" "footprints:Diode-dual"
+		(property "Footprint" "TFL:Diode-dual"
 			(at 118.11 88.9 90)
 			(effects
@@
 			)
 		)
-		(property "Footprint" "footprints:Diode-dual"
+		(property "Footprint" "TFL:Diode-dual"
 			(at 250.19 99.06 90)
 			(effects
@@
 			)
 		)
-		(property "Footprint" "footprints:Diode-dual"
+		(property "Footprint" "TFL:Diode-dual"
 			(at 128.27 64.77 90)
 			(effects
@@
 			)
 		)
-		(property "Footprint" "footprints:Diode-dual"
+		(property "Footprint" "TFL:Diode-dual"
 			(at 158.75 43.18 90)
 			(effects
@@
 			)
 		)
-		(property "Footprint" "footprints:Diode-dual"
+		(property "Footprint" "TFL:Diode-dual"
 			(at 209.55 88.9 90)
 			(effects
@@
 			)
 		)
-		(property "Footprint" "footprints:Diode-dual"
+		(property "Footprint" "TFL:Diode-dual"
 			(at 148.59 64.77 90)
 			(effects
@@
 			)
 		)
-		(property "Footprint" "footprints:Diode-dual"
+		(property "Footprint" "TFL:Diode-dual"
 			(at 158.75 167.64 90)
 			(effects
@@
 			)
 		)
-		(property "Footprint" "footprints:Diode-dual"
+		(property "Footprint" "TFL:Diode-dual"
 			(at 148.59 43.18 90)
 			(effects
@@
 			)
 		)
-		(property "Footprint" "footprints:Diode-dual"
+		(property "Footprint" "TFL:Diode-dual"
 			(at 222.25 167.64 90)
 			(effects
@@
 			)
 		)
-		(property "Footprint" "footprints:Diode-dual"
+		(property "Footprint" "TFL:Diode-dual"
 			(at 209.55 43.18 90)
 			(effects
@@
 			)
 		)
-		(property "Footprint" "footprints:Diode-dual"
+		(property "Footprint" "TFL:Diode-dual"
 			(at 240.03 43.18 90)
 			(effects
@@
 			)
 		)
-		(property "Footprint" "footprints:Diode-dual"
+		(property "Footprint" "TFL:Diode-dual"
 			(at 120.65 167.64 90)
 			(effects
@@
 			)
 		)
-		(property "Footprint" "footprints:Diode-dual"
+		(property "Footprint" "TFL:Diode-dual"
 			(at 179.07 43.18 90)
 			(effects
@@
 			)
 		)
-		(property "Footprint" "footprints:Diode-dual"
+		(property "Footprint" "TFL:Diode-dual"
 			(at 179.07 88.9 90)
 			(effects
@@
 			)
 		)
-		(property "Footprint" "footprints:Diode-dual"
+		(property "Footprint" "TFL:Diode-dual"
 			(at 219.71 88.9 90)
 			(effects
@@
 			)
 		)
-		(property "Footprint" "footprints:Diode-dual"
+		(property "Footprint" "TFL:Diode-dual"
 			(at 212.09 167.64 90)
 			(effects
@@
 			)
 		)
-		(property "Footprint" "footprints:Diode-dual"
+		(property "Footprint" "TFL:Diode-dual"
 			(at 179.07 64.77 90)
 			(effects
@@
 			)
 		)
-		(property "Footprint" "footprints:Diode-dual"
+		(property "Footprint" "TFL:Diode-dual"
 			(at 219.71 43.18 90)
 			(effects
@@
 			)
 		)
-		(property "Footprint" "footprints:Diode-dual"
+		(property "Footprint" "TFL:Diode-dual"
 			(at 265.43 114.3 90)
 			(effects
@@
 			)
 		)
-		(property "Footprint" "footprints:Diode-dual"
+		(property "Footprint" "TFL:Diode-dual"
 			(at 189.23 64.77 90)
 			(effects
@@
 			)
 		)
-		(property "Footprint" "footprints:Diode-dual"
+		(property "Footprint" "TFL:Diode-dual"
 			(at 184.15 167.64 90)
 			(effects
@@
 			)
 		)
-		(property "Footprint" "footprints:Diode-dual"
+		(property "Footprint" "TFL:Diode-dual"
 			(at 130.81 167.64 90)
 			(effects
@@
 			)
 		)
-		(property "Footprint" "footprints:Diode-dual"
+		(property "Footprint" "TFL:Diode-dual"
 			(at 250.19 74.93 90)
 			(effects
@@
 			)
 		)
-		(property "Footprint" "footprints:Diode-dual"
+		(property "Footprint" "TFL:Diode-dual"
 			(at 209.55 64.77 90)
 			(effects
@@
 			)
 		)
-		(property "Footprint" "footprints:Diode-dual"
+		(property "Footprint" "TFL:Diode-dual"
 			(at 118.11 43.18 90)
 			(effects
@@
 			)
 		)
-		(property "Footprint" "footprints:Diode-dual"
+		(property "Footprint" "TFL:Diode-dual"
 			(at 158.75 88.9 90)
 			(effects
@@
 			)
 		)
-		(property "Footprint" "footprints:Diode-dual"
+		(property "Footprint" "TFL:Diode-dual"
 			(at 128.27 43.18 90)
 			(effects
@@
 			)
 		)
-		(property "Footprint" "footprints:Diode-dual"
+		(property "Footprint" "TFL:Diode-dual"
 			(at 118.11 64.77 90)
 			(effects
@@
 			)
 		)
-		(property "Footprint" "footprints:Diode-dual"
+		(property "Footprint" "TFL:Diode-dual"
 			(at 189.23 43.18 90)
 			(effects
@@
 			)
 		)
-		(property "Footprint" "footprints:Diode-dual"
+		(property "Footprint" "TFL:Diode-dual"
 			(at 240.03 64.77 90)
 			(effects
@@
 			)
 		)
-		(property "Footprint" "footprints:Diode-dual"
+		(property "Footprint" "TFL:Diode-dual"
 			(at 250.19 43.18 90)
 			(effects
@@
 			)
 		)
-		(property "Footprint" "footprints:Diode-dual"
+		(property "Footprint" "TFL:Diode-dual"
 			(at 240.03 88.9 90)
 			(effects
@@
 			)
 		)
-		(property "Footprint" "footprints:Diode-dual"
+		(property "Footprint" "TFL:Diode-dual"
 			(at 128.27 88.9 90)
 			(effects
@@
 			)
 		)
-		(property "Footprint" "footprints:Diode-dual"
+		(property "Footprint" "TFL:Diode-dual"
 			(at 219.71 64.77 90)
 			(effects
@@
 			)
 		)
-		(property "Footprint" "footprints:Diode-dual"
+		(property "Footprint" "TFL:Diode-dual"
 			(at 191.77 167.64 90)
 			(effects
