File: QASS_PCB_Zero_lowbar_Germini/QASS_PCB lowbar.kicad_pcb (KiCad board)
At the start: 2 copper layers, 219.1 x 110.5 mm, 104 parts, among them J2 Conn_01x05_Pin, J3 Conn_01x05_Pin, J4 Conn_01x02_Pin, J5 Conn_01x05_Pin, J6 Conn_01x05_Pin, U2 RP2040-Matrix

Commit message: correct version number in Silk
Other:
- board text added: "Re-fork of fork by quark-works: https://github.com/quark-works/QASS-Zero"
- board text added: "v1.3"
- board text removed: "Re-fork of fork by quark-works: https://github.com/quark-works/QASS-Zero - v.1.3"
- board text removed: "v1.2"
Changed lines of the file:
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@@
 		)
 	)
-	(gr_text "v1.2"
+	(gr_text "v1.3"
 		(at 241.5475 22.725625 0)
 		(layer "B.SilkS")
@@
 		)
 	)
-	(gr_text "Re-fork of fork by quark-works: https://github.com/quark-works/QASS-Zero - v.1.3"
+	(gr_text "Re-fork of fork by quark-works: https://github.com/quark-works/QASS-Zero"
 		(at 118.1375 59.865625 0)
 		(layer "B.SilkS")
@@
 			(justify left bottom mirror)
 		)
-		(render_cache "Re-fork of fork by quark-works: https://github.com/quark-works/QASS-Zero - v.1.3"
+		(render_cache "Re-fork of fork by quark-works: https://github.com/quark-works/QASS-Zero"
 			0
 			(polygon
@@
 				)
 			)
-			(polygon
-				(pts
-					(xy 70.682152 59.382994) (xy 70.395167 59.382994) (xy 70.3857 59.38113) (xy 70.37873 59.3759) (xy 70.374162 59.36205)
-					(xy 70.374162 59.315827) (xy 70.376024 59.30639) (xy 70.381243 59.299431) (xy 70.395167 59.294822)
-					(xy 70.682152 59.294822) (xy 70.691615 59.296684) (xy 70.698569 59.301903) (xy 70.703157 59.315827)
-					(xy 70.703157 59.36205) (xy 70.701292 59.371505) (xy 70.696052 59.378451)
-				)
-			)
-			(polygon
-				(pts
-					(xy 69.28374 59.050823) (xy 69.345289 59.050823) (xy 69.356095 59.052777) (xy 69.364912 59.058639)
-					(xy 69.370507 59.067676) (xy 69.584708 59.574358) (xy 69.804527 59.066272) (xy 69.809807 59.057547)
-					(xy 69.817376 59.052589) (xy 69.828279 59.050823) (xy 69.894103 59.050823) (xy 69.903498 59.05266)
-					(xy 69.909372 59.057698) (xy 69.910448 59.073387) (xy 69.90949 59.076103) (xy 69.637892 59.688053)
-					(xy 69.632695 59.696704) (xy 69.625207 59.701636) (xy 69.614139 59.70344) (xy 69.562299 59.70344)
-					(xy 69.550406 59.701304) (xy 69.541646 59.694168) (xy 69.538485 59.688053) (xy 69.268292 59.076103)
-					(xy 69.266192 59.065699) (xy 69.268627 59.057413) (xy 69.274196 59.052717) (xy 69.28289 59.050835)
-				)
-			)
-			(polygon
-				(pts
-					(xy 69.141774 59.707348) (xy 69.108565 59.700046) (xy 69.082703 59.679444) (xy 69.073729 59.664935)
-					(xy 69.068092 59.648295) (xy 69.066181 59.630351) (xy 69.073514 59.596867) (xy 69.094472 59.569894)
-					(xy 69.10891 59.560734) (xy 69.125516 59.555056) (xy 69.141774 59.553353) (xy 69.175217 59.560598)
-					(xy 69.201465 59.581036) (xy 69.210736 59.595472) (xy 69.216626 59.611867) (xy 69.218771 59.630351)
-					(xy 69.216874 59.648215) (xy 69.211406 59.664475) (xy 69.190678 59.690886) (xy 69.176259 59.699858)
-					(xy 69.159582 59.705486)
-				)
-			)
-			(polygon
-				(pts
-					(xy 68.684612 58.710837) (xy 68.713982 58.710837) (xy 68.740605 58.716455) (xy 69.017821 58.827158)
-					(xy 69.026574 58.832088) (xy 69.031195 58.839378) (xy 69.030399 58.85378) (xy 69.015012 58.894386)
-					(xy 69.010094 58.903115) (xy 69.002827 58.907741) (xy 68.988389 58.906964) (xy 68.763014 58.825754)
-					(xy 68.763014 59.67462) (xy 68.761152 59.684083) (xy 68.755933 59.691036) (xy 68.742009 59.695625)
-					(xy 68.684612 59.695625) (xy 68.675119 59.693759) (xy 68.668156 59.68852) (xy 68.663607 59.67462)
-					(xy 68.663607 58.731903) (xy 68.665472 58.722398) (xy 68.670712 58.715411)
-				)
-			)
-			(polygon
-				(pts
-					(xy 68.354335 59.707348) (xy 68.321126 59.700046) (xy 68.295264 59.679444) (xy 68.28629 59.664935)
-					(xy 68.280653 59.648295) (xy 68.278742 59.630351) (xy 68.286075 59.596867) (xy 68.307033 59.569894)
-					(xy 68.321471 59.560734) (xy 68.338077 59.555056) (xy 68.354335 59.553353) (xy 68.387778 59.560598)
-					(xy 68.414026 59.581036) (xy 68.423297 59.595472) (xy 68.429187 59.611867) (xy 68.431332 59.630351)
-					(xy 68.429435 59.648215) (xy 68.423967 59.664475) (xy 68.403239 59.690886) (xy 68.38882 59.699858)
-					(xy 68.372143 59.705486)
-				)
-			)
-			(polygon
-				(pts
-					(xy 67.796606 59.097718) (xy 67.842647 59.10051) (xy 67.842829 59.100527) (xy 67.551631 58.787896)
-					(xy 67.54247 58.769306) (xy 67.5418 58.761273) (xy 67.5418 58.731842) (xy 67.543662 58.722406)
-					(xy 67.548881 58.715446) (xy 67.562805 58.710837) (xy 68.115771 58.710837) (xy 68.125234 58.712699)
-					(xy 68.132187 58.717918) (xy 68.136775 58.731842) (xy 68.136775 58.77947) (xy 68.13491 58.788936)
-					(xy 68.129671 58.795906) (xy 68.115771 58.800474) (xy 67.677599 58.800474) (xy 67.996824 59.142537)
-					(xy 68.002681 59.152353) (xy 68.003545 59.161845) (xy 68.000976 59.170563) (xy 67.992611 59.191568)
-					(xy 67.986459 59.20064) (xy 67.978267 59.204921) (xy 67.964584 59.202803) (xy 67.891822 59.184504)
-					(xy 67.841425 59.180333) (xy 67.801005 59.182277) (xy 67.763958 59.18807) (xy 67.732383 59.196946)
-					(xy 67.703962 59.209106) (xy 67.680049 59.223598) (xy 67.659122 59.240947) (xy 67.641751 59.260464)
-					(xy 67.627334 59.282593) (xy 67.607612 59.334659) (xy 67.600601 59.399053) (xy 67.602537 59.429296)
-					(xy 67.608274 59.457929) (xy 67.617529 59.484374) (xy 67.630261 59.508925) (xy 67.665506 59.551468)
-					(xy 67.713641 59.584748) (xy 67.774726 59.607398) (xy 67.848812 59.617468) (xy 67.865177 59.617772)
-					(xy 67.945827 59.610826) (xy 68.017254 59.591335) (xy 68.078699 59.561861) (xy 68.083592 59.55891)
-					(xy 68.092562 59.554516) (xy 68.100859 59.554861) (xy 68.111618 59.565932) (xy 68.136775 59.616368)
-					(xy 68.139915 59.62888) (xy 68.135899 59.638737) (xy 68.12841 59.644395) (xy 68.082196 59.666926)
-					(xy 68.019094 59.688373) (xy 67.972563 59.698518) (xy 67.919197 59.705216) (xy 67.865177 59.707348)
-					(xy 67.816868 59.70542) (xy 67.771722 59.699737) (xy 67.730744 59.69071) (xy 67.692903 59.678391)
-					(xy 67.658984 59.663296) (xy 67.628177 59.645322) (xy 67.60096 59.62496) (xy 67.576863 59.60207)
-					(xy 67.538434 59.549568) (xy 67.51283 59.488179) (xy 67.50066 59.417941) (xy 67.49979 59.392031)
-					(xy 67.501715 59.352057) (xy 67.507373 59.314847) (xy 67.516389 59.281046) (xy 67.528669 59.249982)
-					(xy 67.543894 59.221935) (xy 67.561999 59.196645) (xy 67.606436 59.154309) (xy 67.661689 59.123042)
-					(xy 67.727724 59.10369)
-				)
-			)
